Commit message: Added collision geometry and improved URDF naming

File: ros2_ws/src/robot_description/urdf/robot.urdf (robot description, URDF)
Before this commit: robot four_axis_robot, 6 links, 5 joints
Links:
- removed link link1
- removed link link2
- removed link link3
- added link bicep_link, mass 10.0; collision box size=0.25 0.045 0.045; visual box size=0.25 0.045 0.045
- added link forearm_link, mass 10.0; collision box size=0.25 0.040 0.040; visual box size=0.25 0.040 0.040
- added link shoulder_link, mass 10.0; collision box size=0.05 0.05 0.25; visual box size=0.05 0.05 0.25
- link base_link: mass None -> 10.0; geometry collision cylinder length=0.10 radius=0.08; visual cylinder length=0.10 radius=0.08
- link tool0: mass None -> 10.0; geometry collision box size=0.15 0.03 0.03; visual box size=0.15 0.03 0.03
Joints:
- removed joint joint1
- removed joint joint2
- removed joint joint3
- removed joint joint4
- added joint base_joint: type revolute, parent base_link, child shoulder_link, origin xyz=0 0 0.125 rpy=0 0 0, axis 0 0 1, limit lower=-3.1416 upper=3.1416 effort=100 velocity=1.0
- added joint elbow_joint: type revolute, parent bicep_link, child forearm_link, origin xyz=0.250 0 0 rpy=0 0 0, axis 0 1 0, limit lower=-1.571 upper=1.571 effort=100 velocity=1.0
- added joint shoulder_joint: type revolute, parent shoulder_link, child bicep_link, origin xyz=0 0 0.250 rpy=0 -1.5708 0, axis 0 1 0, limit lower=-2.094 upper=2.094 effort=100 velocity=1.0
- added joint wrist_joint: type revolute, parent forearm_link, child tool0, origin xyz=0.250 0 0 rpy=0 0 0, axis 0 1 0, limit lower=-1.571 upper=1.571 effort=100 velocity=1.0

Commit message: Update robot URDF with TCP, collision and inertial properties

File: ros2_ws/src/robot_description/urdf/robot.urdf (robot description, URDF)
Before this commit: robot four_axis_robot, 6 links, 5 joints
Links:
- link tcp: mass None -> 0.1
